File: bkm-129x-simple.sch (KiCad schematic (older format))
At the start: 55 parts, among them J1 YG_IN, J11 YG_OUT, J2 PBB_IN, J21 PBB_OUT, J3 PRR_IN, J31 PRR_OUT, J4 SYNC_IN, J41 SYNC_OUT, J5 Conn_02x32_Row_Letter_Last, Q1 DTC144EKA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

Commit message: Rev B: Added onboard MCU
Connections:
- net ~MCU_SS: now reaches U3.13 (14/PB2/OC1B/PCINT2/~SS), U4.1 (E), U4.10 (E), U4.11 (O), U4.4 (E)
- net MCU_MOSI: now reaches U3.14 (15/PB3/OC2/PCINT3/MOSI), U4.8 (O)
- net MCU_MISO: now reaches R23.1, U3.15 (16/PB4/PCINT4/MISO), U4.5 (D)
- no-connect marks 38 -> 40
Other:
- moved on the sheet: R19
Changed lines of the file:
@@
 $Descr A4 11693 8268
 encoding utf-8
-Sheet 1 1
-Title ""
-Date ""
-Rev ""
+Sheet 1 2
+Title "BKM-129X Compatible full size"
+Date "2020-07-27"
+Rev "B"
 Comp ""
 Comment1 ""
@@
 	0    -1   -1   0
 $EndComp
-Text Label 6500 5050 0    60   ~ 0
-~MCU_RESET
 NoConn ~ 6500 4750
 NoConn ~ 6500 5350
@@
 NoConn ~ 6500 6700
 NoConn ~ 3700 5050
-Text Label 3700 5350 2    60   ~ 0
-MCU_SLOT_ID
 $Comp
 L DTC144EKA Q1
@@
 	1    0    0    -1
 $EndComp
-Text Label 8350 5150 2    60   ~ 0
-~MCU_RESET
-Wire Wire Line
-	8350 5150 8500 5150
 Connection ~ 8500 5150
 $Comp
@@
 	750  6900 800  6900
 Connection ~ 750  6900
-Wire Wire Line
-	1150 6900 1150 6800
 Connection ~ 1150 6900
 $Comp
@@
 Wire Wire Line
 	1300 6100 1400 6100
-Text Label 1150 6800 1    60   ~ 0
-MCU_SLOT_ID
 Text Label 750  7100 3    60   ~ 0
 SLOT_ID
@@
 Wire Wire Line
 	1300 4600 1400 4600
-Text Label 2300 4600 0    60   ~ 0
-MCU_SCK
-Text Label 6500 6850 0    60   ~ 0
-MCU_SCK
 $Comp
 L CP C8
@@
 L R R19
 U 1 1 5E4AFA4C
-P 3050 4750
-F 0 "R19" V 3130 4750 50  0000 C CNN
-F 1 "4K7" V 3050 4750 50  0000 C CNN
-F 2 "Resistors_SMD:R_0805_HandSoldering" V 2980 4750 50  0001 C CNN
-F 3 "" H 3050 4750 50  0001 C CNN
-	1    3050 4750
+P 3050 4550
+F 0 "R19" V 3130 4550 50  0000 C CNN
+F 1 "4K7" V 3050 4550 50  0000 C CNN
+F 2 "Resistors_SMD:R_0805_HandSoldering" V 2980 4550 50  0001 C CNN
+F 3 "" H 3050 4550 50  0001 C CNN
+	1    3050 4550
 	-1   0    0    1
 $EndComp
@@
 L +5VD #PWR060
 U 1 1 5E4AFB1C
-P 3050 4600
-F 0 "#PWR060" H 3050 4450 50  0001 C CNN
-F 1 "+5VD" H 3050 4750 50  0000 C CNN
-F 2 "" H 3050 4600 50  0001 C CNN
-F 3 "" H 3050 4600 50  0001 C CNN
-	1    3050 4600
-	1    0    0    -1
-$EndComp
-Text Label 3050 4900 3    60   ~ 0
-MCU_SCK
+P 3050 4400
+F 0 "#PWR060" H 3050 4250 50  0001 C CNN
+F 1 "+5VD" H 3050 4550 50  0000 C CNN
+F 2 "" H 3050 4400 50  0001 C CNN
+F 3 "" H 3050 4400 50  0001 C CNN
+	1    3050 4400
+	1    0    0    -1
+$EndComp
 $Comp
 L MIC3490 U5
@@
 	0    1    1    0
 $EndComp
+$Sheet
+S 3450 3700 1100 650
+U 5F1F170D
+F0 "Onboard-MCU" 60
+F1 "atmega328p.sch" 60
+$EndSheet
+Text GLabel 8350 5150 0    60   Input ~ 0
+~MCU_RESET
+Text GLabel 6500 5050 2    60   Input ~ 0
+~MCU_RESET
+Wire Wire Line
+	8350 5150 8500 5150
+Text GLabel 2300 4600 2    60   Input ~ 0
+MCU_SCK
+Text GLabel 6500 6850 2    60   Input ~ 0
+MCU_SCK
+Text GLabel 3050 4700 3    60   Input ~ 0
+MCU_SCK
+Text GLabel 1150 7000 3    60   Input ~ 0
+MCU_SLOT_ID
+Text GLabel 3600 5350 0    60   Input ~ 0
+MCU_SLOT_ID
+Wire Wire Line
+	1150 7000 1150 6900
+Wire Wire Line
+	3600 5350 3700 5350
+Text GLabel 3100 6950 3    60   Input ~ 0
+~MCU_SS
+Text GLabel 3300 6950 3    60   Input ~ 0
+MCU_MOSI
+Text GLabel 3500 6950 3    60   Input ~ 0
+MCU_MISO
+Wire Wire Line
+	3100 6950 3100 6550
+Connection ~ 3100 6550
+Wire Wire Line
+	3300 6950 3300 6700
+Connection ~ 3300 6700
+Wire Wire Line
+	3500 6950 3500 6850
+Connection ~ 3500 6850
+NoConn ~ 3700 4750
+NoConn ~ 3700 4900
 $EndSCHEMATC

Commit message: Fixed the THS7374 filter stuff, moved to Kicad 5
Parts:
- C1, C10, C11, C12, C2, C3, C4, C5, C6, C9: symbol C -> bkm-129x-simple-rescue:C
- C13, C7, C8: symbol CP -> bkm-129x-simple-rescue:CP
- J1, J11, J2, J21, J3, J31, J4, J41: symbol Conn_Coaxial -> bkm-129x-simple-rescue:Conn_Coaxial
- J5: symbol Conn_02x32_Row_Letter_Last -> bkm-129x-simple-rescue:Conn_02x32_Row_Letter_Last
- Q1: symbol DTC144EKA -> dtc144eka:DTC144EKA
- R1, R10, R11, R12, R13, R18, R19, R20, R21, R22, R23, R24, R25, R26, R27, R28, R29, R30, R31, R6, R7, R8, R9: symbol R -> bkm-129x-simple-rescue:R
- SW1, SW2, SW3, SW4: symbol SW_DPDT_x2 -> bkm-129x-simple-rescue:SW_DPDT_x2
- U1: symbol ADG1611 -> adg1611:ADG1611
- U2: symbol THS7374 -> ths7374:THS7374
- U3: symbol arduino-nano-v3 -> arduino-nano-v3:arduino-nano-v3
- U4: symbol 74LVC125 -> bkm-129x-simple-rescue:74LVC125
- U5: symbol MIC3490 -> mic3490:MIC3490
Connections:
- net +3V3: now also U2.9 (BYPASS)
- net GND: no longer U2.9 (BYPASS)

Commit message: Revision D
Parts:
- added C101: 1uF, Capacitor_SMD:C_0805_2012Metric_Pad1.18x1.45mm_HandSolder, symbol bkm-129x-simple-rescue:C
- added C102: 4.7uF, Capacitor_SMD:C_0805_2012Metric_Pad1.18x1.45mm_HandSolder, symbol bkm-129x-simple-rescue:C
- added U101: LD1117S33TR_SOT223, Package_TO_SOT_SMD:SOT-223-3_TabPin2, symbol Regulator_Linear:LD1117S33TR_SOT223
- C1, C10, C11, C12, C2, C3, C4, C5, C6, C9: footprint Capacitors_SMD:C_0805_HandSoldering -> Capacitor_SMD:C_0805_2012Metric_Pad1.18x1.45mm_HandSolder
- C13, C7, C8: footprint Capacitors_SMD:CP_Elec_6.3x5.3 -> Capacitor_SMD:CP_Elec_6.3x5.3
- J5: footprint din-41612-64p-ra:DIN-41612-64P -> standard-pin-64p-ra:STANDARD-PIN-64P-RA
- Q1: footprint TO_SOT_Packages_SMD:SC-59_Handsoldering -> Package_TO_SOT_SMD:SC-59_Handsoldering
- R1, R10, R11, R12, R13, R18, R19, R20, R21, R22, R23, R24, R25, R26, R27, R28, R29, R30, R31, R6, R7, R8, R9: footprint Resistors_SMD:R_0805_HandSoldering -> Resistor_SMD:R_0805_2012Metric_Pad1.20x1.40mm_HandSolder
- U1: footprint Housings_SSOP:TSSOP-16_4.4x5mm_Pitch0.65mm -> Package_SO:TSSOP-16_4.4x5mm_P0.65mm
- U2, U4: footprint Housings_SSOP:TSSOP-14_4.4x5mm_Pitch0.65mm -> Package_SO:TSSOP-14_4.4x5mm_P0.65mm
- U5: footprint TO_SOT_Packages_SMD:SOT-23-5_HandSoldering -> Package_TO_SOT_SMD:SOT-23-5_HandSoldering
Connections:
- net +3V3: now also C102.1, U101.2 (VO)
- net GND: now also C101.2, C102.2, U101.1 (GND)
- net VDD: now also C101.1, U101.3 (VI)
Other:
- moved on the sheet: C10, C11, U5
